File: MainPCB/EnvKB110ADR.sch (KiCad schematic (older format))
At the start: 246 parts, among them U1 MCP23017_SO, U2 Pico

Commit message: Added Logo and couple small corrections to traces.
Parts:
- U1: value MCP23017_SO -> MCP23017; LCSC (none) -> MCP23017_SO
Changed lines of the file:
@@
 P 15700 13450
 F 0 "U1" H 15700 14731 50  0000 C CNN
-F 1 "MCP23017_SO" H 16100 14600 50  0000 C CNN
+F 1 "MCP23017" H 16100 14600 50  0000 C CNN
 F 2 "Package_SO:SOIC-28W_7.5x17.9mm_P1.27mm" H 15900 12450 50  0001 L CNN
 F 3 "http://ww1.microchip.com/downloads/en/DeviceDoc/20001952C.pdf" H 15900 12350 50  0001 L CNN
+F 4 "MCP23017_SO" H 15700 13450 50  0001 C CNN "LCSC"
 	1    15700 13450
 	1    0    0    -1
