File: MainPCB/EnvKB110ADR.kicad_pcb (KiCad board)
At the start: 2 copper layers, 429.5 x 133.3 mm, 246 parts, among them U1 MCP23017_SO, U2 Pico

Commit message: Added Logo and couple small corrections to traces.
Routing:
- net col14: track 248.6 -> 250.1 mm
Other:
- board text added: "https://github.com/Envious-Data/Env-KB110ADR"

Commit message: whatamidoing
Routing:
- net row0: track 321.4 -> 326.9 mm
- net col4: track 439.7 -> 444.9 mm
- net col22: track 116.0 -> 121.2 mm
- net col3: track 487.9 -> 492.6 mm
- net col1: track 501.4 -> 505.7 mm
- net col0: track 529.4 -> 533.5 mm
- net SDA: track 78.6 -> 81.2 mm
- net row1: track 358.3 -> 360.8 mm
- net col6: track 392.9 -> 395.3 mm
- net col2: track 485.8 -> 488.1 mm
- net SCL: track 74.7 -> 76.9 mm
- net col5: track 415.7 -> 417.9 mm
- net col15: track 185.9 -> 183.9 mm
- net col14: track 250.1 -> 252.0 mm
- net col7: track 386.4 -> 387.9 mm
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